File: kicad/mobile-antenna-switch.kicad_sch (KiCad schematic)
At the start: 54 parts

Commit message: more schematic and sim work
Parts:
- removed U? (x2): TC4428VOA, symbol TC442x:TC4428VOA
- removed U? (x2): MASW-000936, symbol MACOM_MASW:MASW-000936
- added C19: 10uF, symbol Device:C_Small
- added F1: 500mA, symbol Device:Polyfuse_Small
- added J?: Conn_01x04_Female, symbol Connector:Conn_01x04_Female
- added U1, U3: TC4428VOA, symbol TC442x:TC4428VOA
- added U2, U4: MASW-000936, Package_DFN_QFN:QFN-16-1EP_4x4mm_P0.65mm_EP2.5x2.5mm_ThermalVias, symbol MACOM_MASW:MASW-000936
- C1, C10, C11, C12, C13, C14, C16, C17, C18, C2, C3, C4, C5, C7, C8, C9: renamed from C?; value 68pF -> 180pF
- L1, L2, L3, L4, L5, L6, L7, L8: renamed from L?; value 1uH -> 100nH
- gave numbers to parts that had none: 26
Connections:
- net +12V: now also C19.1, F1.1, U1.6 (VDD), U3.6 (VDD)
- net GND: now also C19.2, J?.4 (Pin_4), U1.3 (GND), U2.1 (GND), U2.11 (GND), U2.13 (GND), U2.17 (EP), U2.8 (GND), U3.3 (GND), U4.1 (GND), U4.11 (GND), U4.13 (GND), U4.17 (EP), U4.8 (GND)
- net ~{EN}: now also U1.2 (INA), U1.4 (INB), U3.2 (INA), U3.4 (INB)
- net at C17.1, L6.1: now also U4.14 (TX)
- net at C18.1, L7.2: now also U4.7 (RX)
- net at C9.1, L3.2: now also U2.7 (RX)
- net at C8.1, L2.1: now also U2.14 (TX)
- net at C2.2, L1.2: now also U2.2 (ANT)
- net at C11.2, L5.2: now also U4.2 (ANT)
- net at L8.1: now also U4.9 (RXB)
- net at L4.1: now also U2.9 (RXB)
- net RX renamed RX1
- net RX1: now also U1.7 (~{OUTA}); no longer R16.2
- net TX renamed TX1
- net TX1: now also U1.5 (OUTB); no longer R15.2, R18.2
- new net: F1.2, J?.1 (Pin_1)
- new net RX2: R16.2, U3.7 (~{OUTA})
- new net TX2: R15.2, R18.2, U3.5 (OUTB)
- new net ~{PTT_IN}: J?.2 (Pin_2)
- new net ~{PTT_OUT}: J?.3 (Pin_3)
Other:
- moved on the sheet: C1, C10, C11, C2, J1, J4, L1, L5, R1, R10, R11, R14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

Commit message: more schematic and sim work
Parts:
- added Q?: Q_PMOS_GSD, symbol Device:Q_PMOS_GSD
- added Q?: Q_NMOS_GSD, symbol Device:Q_NMOS_GSD
- added R? (x2): 10k, symbol Device:R_Small
- added U?: LM556, symbol Timer:LM556
Connections:
- net +12V: now also Q?.3 (D), R?.1
- net GND: now also Q?.2 (S), R?.2
- net ~{PTT_IN}: now also Q?.1 (G), R?.2
- net ~{PTT_OUT}: now also Q?.3 (D)
- new net: Q?.1 (G), Q?.2 (S), R?.1
